File: Hardware/Proiect_TSC_schema.sch (EAGLE design)
At the start: 103 parts, among them IC1 BD5229G-TR, IC4 XC6220A331MR-G, J1 FH34SRJ-24S-0.5SH_99_, J2 SAMACSYS_PARTS_USB4110-GF-A, J3 QWIIC_RIGHT_ANGLE, J4 112A-TAAR-R03_ATTEND, Q1 20V/4.2A/52mΩ/1.4W, Q2 20V/4.2A/52mΩ/1.4W, Q3 SI1308EDL-T1-GE3, U1 W25Q512JVEIQ, U2 ESP32-C6-WROOM-1-N8, U3 DS3231SN#, U4 MAX17048G+T10, U5 ESP32_WROVER_SPARKFUN-IC-POWE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

Commit message: Update schematic and PCB
Parts:
- R_CAPACITOR: value (none) -> 15
- renumbered TP1 to TX, TP10 to EPD_CS, TP16 to 3V3, TP17 to EPD_3V3, TP2 to RX, TP3 to VBAT, TP4 to GND, TP5 to GND_TP5, TP6 to MISO, TP7 to MOSI, TP8 to SCK, TP9 to EPD_BUSY
Connections:
- removed net N$10: J1.MP1, J1.MP2
- removed net N$13: EPD_C1.1, EPD_C2.1, J1.8
- removed net N$18: R_RESET.2
- removed net N$20: Q2.D
- removed net N$26: U3.GND
- removed net N$5 (its old number): SJ1.1
- removed net N$8: R4.1
- net 3V3: now also Q2.D, R_RESET.2
- net GND: now also EPD_C1.1, EPD_C2.1, J1.8, J1.MP1, J1.MP2, R4.1, SJ1.1, U3.GND
